File: PWMs/Hall Effect/PWM Module 3.0A.kicad_sch (KiCad schematic)
At the start: 4 parts, among them J1 PH1-20-UA, J2 PH1-20-UA

Commit message: HEffect KiCad
Parts:
- added opamp1: ADA4510-2ARZ, R-8_ADI, symbol Project-Syms:ADA4510-2ARZ
- R1: value 2k -> 3k
- R2: value 6k -> 2k
Connections:
- net GND: no longer J1.15
- net Hall Effect Out: now also J2.4, R2.1; no longer J2.15, R1.1
- net V(2.5V): now also opamp1.3 (INA+)
- net Vout+: now also J2.5, R1.1, opamp1.1 (OUTA); no longer J2.8, R2.2
- net at J1.2: now also opamp1.4 (V-)
- net +5V in: now reaches J1.3
- net +5V in: now also opamp1.8 (V+)
- net at R1.2: now also R2.2, opamp1.2 (INA-); no longer R2.1
