File: PWMs/Hall Effect/PWM Module 3.0A.kicad_pcb (KiCad board)
At the start: 2 copper layers, 50.5 x 46 mm, 4 parts, among them J1 PH1-20-UA, J4 PH1-20-UA

Commit message: HEffect KiCad
Parts:
- removed J4: PH1-20-UA, Connector_PinHeader_2.54mm:PinHeader_1x20_P2.54mm_Vertical
- added J2: PH1-20-UA, Connector_PinHeader_2.54mm:PinHeader_1x20_P2.54mm_Vertical, F.Cu at (152.4, 25.4)
- added opamp1: ADA4510-2ARZ, Project-PCB-Syms.bak:R-8_ADI, F.Cu at (177.8, 48.3)
- R1: value 2k -> 3k
- R2: value 6k -> 2k
- moved J1 43.2 mm to (152.4, 68.6)
- moved R1 14.1 mm to (165.1, 53.3), turned to 90 degrees
- moved R2 1.20 mm to (157.5, 53.3), turned to 90 degrees
Connections:
- J1 pad 15: GND -> unconnected-(J1-Pad15)
- J1 pad 2: unconnected-(J1-Pad2) -> Net-(opamp1-V-)
- J1 pad 3: unconnected-(J1-Pad3) -> +5V in
- R1 pad 1: Hall Effect Out -> Vout+
- R1 pad 2: Net-(U1--) -> Net-(opamp1-INA-)
- R2 pad 1: Net-(U1--) -> Hall Effect Out
- R2 pad 2: Vout+ -> Net-(opamp1-INA-)
Routing:
- net V(2.5V): track 0.00 -> 71.3 mm
- net Vout+: track 6.64 -> 77.2 mm
- net +5V in: track 0.00 -> 58.2 mm
- net Net-(opamp1-INA-): track 0.00 -> 56.7 mm
- net Net-(opamp1-V-): track 0.00 -> 41.3 mm
- net Hall Effect Out: track 0.00 -> 39.2 mm
- net Net-(U1--): track 17.8 -> 0.00 mm
Other:
- board text added: "15"
- board text added: "19"
- board text added: "24: H-effect 25: Vout"
- board text added: "2: GND 3: 5V+ 23: 2.5V+"
- board text added: "5"
- board text removed: "3: VCU Fan 4: VCU Pump 5: 5V+ Supply"

Commit message: add pin marker
Other:
- board text added: "25"
- board text added: "30"
Changed lines of the file:
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@@
+		)
+	)
+	(gr_text "25"
+		(at 162.56 27.94 0)
+		(layer "User.1")
+		(effects
+			(font
+				(size 0.5 0.5)
+				(thickness 0.125)
+				(bold yes)
+			)
+			(justify left bottom)
+		)
+	)
+	(gr_text "30"
+		(at 175.26 27.94 0)
+		(layer "User.1")
+		(effects
+			(font
+				(size 0.5 0.5)
+				(thickness 0.125)
+				(bold yes)
+			)
+			(justify left bottom)
 		)
 	)
