File: PWMs & Hall Effect Sensor/Hall Effect Sensor/Hall Effect Sensor.kicad_sch (KiCad schematic)
At the start: 7 parts, among them J1 PH1-20-UA, J2 PH1-20-UA

Commit message: Moved folders around
Changed the op amp to a very similar one that can handle a 5V supply
Parts:
- opamp1: symbol Project-Syms:ADA4510-2ARZ -> Project-Syms:ADA4522-2ARZ-RL
Changed lines of the file:
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@@
 	)
 	(symbol
-		(lib_id "Project-Syms:ADA4510-2ARZ")
+		(lib_id "Project-Syms:ADA4522-2ARZ-RL")
 		(at 50.8 90.17 0)
 		(unit 1)
@@
 			)
 		)
-		(property "Datasheet" "ADA4510-2ARZ"
+		(property "Datasheet" "https://www.analog.com/media/en/technical-documentation/data-sheets/ADA4522-1_4522-2_4522-4.pdf"
 			(at 50.8 90.17 0)
 			(effects
