File: PWMs & Hall Effect Sensor/Hall Effect Sensor/Hall Effect Sensor.kicad_pcb (KiCad board)
At the start: 2 copper layers, 50.5 x 46 mm, 7 parts, among them J1 PH1-20-UA, J2 PH1-20-UA

Commit message: Shrunk Hall Effect
Parts:
- removed J2: PH1-20-UA, Connector_PinHeader_2.54mm:PinHeader_1x20_P2.54mm_Vertical
- added J1: PH1-20-UA, Connector_PinHeader_2.54mm:PinHeader_1x20_P2.54mm_Vertical, F.Cu at (152.9, 26.2)
Other:
- board size 50.5 x 46 mm -> 34.9 x 46 mm
