File: Circuit Power Module/Circuit Power Module V2.0/Circuit Power Module.kicad_sch (KiCad schematic)
At the start: 7 parts, among them J1 VBATT +, J2 Vs

Commit message: Renaming stuff on boards that was wrong
RTDS schematic was totally totally wrong with the pins compared to the PCB
Changed lines of the file:
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@@
 (kicad_sch
-	(version 20231120)
+	(version 20250114)
 	(generator "eeschema")
-	(generator_version "8.0")
+	(generator_version "9.0")
 	(paper "A4")
 	(junction
@@
 		(dnp no)
 		(property "Reference" "J2"
-			(at 149.606 50.8 90)
+			(at 149.606 53.594 90)
 			(effects
 				(font
@@
 		)
 		(property "Value" "Vs"
-			(at 149.86 53.3399 90)
+			(at 149.86 50.8 90)
 			(effects
 				(font
@@
 		)
 	)
+	(embedded_fonts no)
 )
