File: I-O Board/IO Module V2.0/IO Module V2.0.kicad_sch (KiCad schematic)
At the start: 18 parts, among them J1 PH1-10-UA, J10 691137710002, J11 691137710002, J2 *, J3 *, J4 *, J5 20-0600-21, J6 20-0600-21, J7 691137710002, J8 691137710002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

Commit message: Renaming stuff on boards that was wrong
RTDS schematic was totally totally wrong with the pins compared to the PCB
Parts:
- renumbered J5 to J2, J6 to J4
Other:
- note added: "From Charge Enable Switch"
- note added: "Unused"
- note removed: "Driver Input 0"
- note removed: "Driver Input 1"
- note removed: "Driver Input 2"
- note removed: "Driver Input 3"
- note removed: "VCU Charge Enable (12V)"
