File: VCU Charge Status/VCU Charge Mode Signal Module V3.1/VCU Charge Mode Signal Module V3.1.kicad_pcb (KiCad board)
At the start: 2 copper layers, 46 x 25 mm, 6 parts, among them J1 PH1-10-UA, J2 PH1-10-UA, U1 IRLML2060TRPBF

Commit message: Renaming stuff on boards that was wrong
RTDS schematic was totally totally wrong with the pins compared to the PCB
Other:
- board text added: "1: +5V 3: GND 2: From CE Switch 4: CE-5V"
- board text added: "VCU Charge Mode Signal Module V3.1 | J.W. Sep '25"
- board text removed: "1: +5V 3: GND 2: CE-12V 4: CE-5V"
- board text removed: "VCU Charge Mode Signal Module V3.1 | J.W. Mar '25"
