File: I-O Board/I-O Board V3.0/I-O Board V3.0.kicad_pcb (KiCad board)
At the start: 2 copper layers, 58.1 x 146.2 mm, 24 parts, among them J1 PH1-10-UA, J10 691137710002, J11 691137710002, J2 *, J3 *, J4 *, J5 B12B-PH-K-S, J6 20-0600-21, J6 B12B-PH-K-S, J7 691137710002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

Commit message: IO board V3.0 fully done?
Parts:
- removed the J6 at (101.0, 75.5)
- removed mounting hole 1: MountingHole_3.5mm, MountingHole:MountingHole_3.5mm
- removed mounting hole 2: MountingHole_3.5mm, MountingHole:MountingHole_3.5mm
- removed mounting hole 3: MountingHole_3.5mm, MountingHole:MountingHole_3.5mm
- added J12: Conn_01x15, Connector_JST:JST_PH_B15B-PH-K_1x15_P2.00mm_Vertical, F.Cu at (88.0, 74.5)
- added J13: Conn_01x15, Connector_JST:JST_PH_B15B-PH-K_1x15_P2.00mm_Vertical, F.Cu at (99.6, 74.0)
- J5: value B12B-PH-K-S -> Conn_01x15; footprint MotorSports_KICad:CONN12_B12B-PH_JST -> Connector_JST:JST_PH_B15B-PH-K_1x15_P2.00mm_Vertical
- moved J9 119.6 mm to (102.5, 148.5), turned to 0 degrees
- moved F1 116.2 mm to (91.0, 36.3), turned to 0 degrees
- moved J11 111.9 mm to (104.6, 27.1), turned to 0 degrees
- moved J8 104.4 mm to (89.5, 148.5), turned to 0 degrees
- moved J7 83.0 mm to (86.5, 27.0), turned to 0 degrees
- moved J10 76.7 mm to (106.0, 46.9), turned to 0 degrees
- moved R28 43.6 mm to (61.5, 158.5), turned to 0 degrees
- moved R29 43.0 mm to (61.6, 152.8), turned to 180 degrees
- moved R26 39.4 mm to (85.6, 120.9)
- moved R23 35.5 mm to (85.6, 125.0)
- moved R31 28.6 mm to (73.2, 158.5), turned to 0 degrees
- moved R30 28.1 mm to (73.2, 152.9), turned to 0 degrees
- moved J2 3.36 mm to (77.3, 48.2)
- moved J3 1.69 mm to (77.3, 88.5)
- moved J5 1.07 mm to (112.5, 74.5)
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- renumbered J6 to J12
Connections:
- J12 pad 1: unconnected-(J6-Pad1) -> (no net)
- J12 pad 13: unconnected-(J6-Pad13) -> (no net)
- J12 pad 14: unconnected-(J6-Pad14) -> (no net)
- J12 pad 15: unconnected-(J6-Pad15) -> (no net)
- J12 pad 16: unconnected-(J6-Pad16) -> (no net)
- J12 pad 17: unconnected-(J6-Pad17) -> (no net)
- J12 pad 18: unconnected-(J6-Pad18) -> (no net)
- J12 pad 19: unconnected-(J6-Pad19) -> (no net)
- J12 pad 20: unconnected-(J6-Pad20) -> (no net)
- J12 pad 3: unconnected-(J6-Pad3) -> (no net)
- J2 pad 05: unconnected-(J2-Pad05) -> Net-(J5-Pin_5)
- J2 pad 06: Net-(J2-Pad06) -> Net-(J5-Pin_6)
- J2 pad 07: Net-(J2-Pad07) -> Net-(J5-Pin_7)
- J2 pad 08: Net-(J2-Pad08) -> Net-(J5-Pin_8)
- J2 pad 09: Net-(J2-Pad09) -> Net-(J5-Pin_9)
- J2 pad 10: Net-(J2-Pad10) -> Net-(J5-Pin_10)
- J2 pad 11: Net-(J2-Pad11) -> Net-(J5-Pin_11)
- J2 pad 12: Net-(J2-Pad12) -> Net-(J5-Pin_12)
- J2 pad 13: Net-(J2-Pad13) -> Net-(J5-Pin_13)
- J2 pad 14: Net-(J2-Pad14) -> Net-(J5-Pin_14)
- J2 pad 15: Net-(J2-Pad15) -> Net-(J5-Pin_15)
- J3 pad 01: unconnected-(J3-Pad01) -> Net-(J12-Pin_1)
- J3 pad 02: unconnected-(J3-Pad02) -> Net-(J12-Pin_2)
- J3 pad 03: unconnected-(J3-Pad03) -> Net-(J12-Pin_3)
- J3 pad 04: unconnected-(J3-Pad04) -> Net-(J12-Pin_4)
- J3 pad 05: unconnected-(J3-Pad05) -> Net-(J12-Pin_5)
- J3 pad 06: unconnected-(J3-Pad06) -> Net-(J12-Pin_6)
- J3 pad 07: unconnected-(J3-Pad07) -> Net-(J12-Pin_7)
- J3 pad 08: unconnected-(J3-Pad08) -> Net-(J12-Pin_8)
- J3 pad 09: unconnected-(J3-Pad09) -> Net-(J12-Pin_9)
- J3 pad 10: unconnected-(J3-Pad10) -> Net-(J12-Pin_10)
- J3 pad 11: unconnected-(J3-Pad11) -> Net-(J12-Pin_11)
- J4 pad 02: unconnected-(J4-Pad02) -> Net-(J13-Pin_1)
- J4 pad 03: unconnected-(J4-Pad03) -> Net-(J13-Pin_3)
- J5 pad 10: Net-(J2-Pad11) -> Net-(J5-Pin_10)
- J5 pad 11: Net-(J2-Pad12) -> Net-(J5-Pin_11)
- J5 pad 12: Net-(J2-Pad13) -> Net-(J5-Pin_12)
- J5 pad 5: Net-(J2-Pad06) -> Net-(J5-Pin_5)
- J5 pad 6: Net-(J2-Pad07) -> Net-(J5-Pin_6)
- J5 pad 7: Net-(J2-Pad08) -> Net-(J5-Pin_7)
- J5 pad 8: Net-(J2-Pad09) -> Net-(J5-Pin_8)
- J5 pad 9: Net-(J2-Pad10) -> Net-(J5-Pin_9)
Routing:
- net Net-(J5-Pin_9): track 0.00 -> 71.1 mm
- net Net-(J5-Pin_10): track 0.00 -> 70.7 mm
- net Net-(J5-Pin_11): track 0.00 -> 70.1 mm
- net Net-(J5-Pin_12): track 0.00 -> 70.0 mm
- net Net-(J5-Pin_13): track 0.00 -> 69.9 mm
- net Net-(J5-Pin_14): track 0.00 -> 68.9 mm
- net Net-(J2-Pad09): track 68.9 -> 0.00 mm
- net Net-(J2-Pad10): track 68.6 -> 0.00 mm
- net Net-(J5-Pin_15): track 0.00 -> 68.5 mm
- net Net-(J2-Pad11): track 67.3 -> 0.00 mm
- net Net-(J2-Pad12): track 66.7 -> 0.00 mm
- net Net-(J2-Pad13): track 65.5 -> 0.00 mm
- net unconnected-(J4-Pad02): track 63.1 -> 0.00 mm
- net Net-(J13-Pin_1): track 0.00 -> 62.7 mm
- net Net-(J13-Pin_3): track 0.00 -> 55.6 mm
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Other:
- board text added: "J12-1"
- board text added: "J12-10"
- board text added: "J12-11"
- board text added: "J12-12"
- board text added: "J12-13"
- board text added: "J12-14"
- board text added: "J12-2"
- board text added: "J12-3"
- board text added: "J12-4"
- board text added: "J12-5"
- board text added: "J12-6"
- board text added: "J12-7"
- board text added: "J12-8"
- board text added: "J12-9"
- board text added: "J13-1"
- board text added: "J13-10"
- board text added: "J13-11"
- board text added: "J13-12"
- board text added: "J13-13"
- board text added: "J13-14"
- board text added: "J13-15"
- board text added: "J13-2"
- board text added: "J13-3"
- board text added: "J13-4"
- board text added: "J13-5"
- board text added: "J13-6"
- board text added: "J13-7"
- board text added: "J13-8"
- board text added: "J13-9"
- board text added: "J5-1"
- board text added: "J5-10"
- board text added: "J5-11"
- board text added: "J5-12"
- board text added: "J5-13"
- board text added: "J5-14"
- board text added: "J5-15"
- board text added: "J5-2"
- board text added: "J5-3"
- board text added: "J5-4"
- board text added: "J5-5"
- board text added: "J5-6"
- board text added: "J5-7"
- board text added: "J5-8"
- board text added: "J5-9"
- board text added: "Wrong Side flip over"
