File: I-O Board/I-O Board V3.0/_autosave-I-O Board V3.0.kicad_sch (KiCad schematic)
At the start: 19 parts, among them J1 PH1-10-UA, J10 691137710002, J11 691137710002, J13 691137710002, J2 *, J3 *, J4 *, J5 Conn_01x15, J6 Conn_01x15, J7 Conn_01x15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

Commit message: IO board V3.0 fully done?
Changed lines of the file:
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@@
-		)
-	)
-	(text "AMS LED +"
-		(exclude_from_sim no)
-		(at 98.552 14.224 0)
-		(effects
-			(font
-				(size 1.27 1.27)
-			)
 		)
 	)
