File: RTDSPrecharge/RTDSPrecharge/RTDSPrecharge.kicad_sch (KiCad schematic)
At the start: 34 parts, among them J1 PH1-10-UA, K1 G6L-1P_DC5, Q1 SS8550, U1 NE555D, U2 IRLML2060TRPBF, U3 IRLML2060TRPBF, U4 IRLML2060TRPBF, U5 PMV160UP, U6 NE555D, U7 IRLML2060TRPBF

Commit message: documentation
documentation
Other:
- note added: "Precharge"
- note added: "RTDS"
Changed lines of the file:
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@@
 	(generator_version "9.0")
 	(paper "A4")
+	(rectangle
+		(start 41.91 101.6)
+		(end 261.62 170.18)
+		(stroke
+			(width 0)
+			(type default)
+		)
+		(fill
+			(type none)
+		)
+	)
+	(rectangle
+		(start 43.18 49.53)
+		(end 186.69 99.06)
+		(stroke
+			(width 0)
+			(type default)
+		)
+		(fill
+			(type none)
+		)
+	)
 	(text "RTDS Coil -\n"
 		(exclude_from_sim no)
@@
 			(font
 				(size 0.762 0.762)
+			)
+		)
+	)
+	(text "RTDS"
+		(exclude_from_sim no)
+		(at 48.514 47.752 0)
+		(effects
+			(font
+				(size 1.27 1.27)
 			)
 		)
@@
 		(effects
 			(font
+				(size 1.27 1.27)
+			)
+		)
+	)
+	(text "Precharge\n"
+		(exclude_from_sim no)
+		(at 45.466 172.974 0)
+		(effects
+			(font
