File: RTDSPrecharge/RTDSPrecharge/RTDSPrecharge.kicad_pcb (KiCad board)
At the start: 2 copper layers, 74.5 x 77 mm, 34 parts, among them J1 PH1-10-UA, K1 G6L-1P_DC5, Q1 SS8550, U1 NE555D, U2 IRLML2060TRPBF, U3 IRLML2060TRPBF, U4 IRLML2060TRPBF, U5 PMV160UP, U6 NE555D, U7 IRLML2060TRPBF

Commit message: Silkscreen
silkscreen
Other:
- board text added: "RTDS-Precharge | H.R. Oct '28"
Changed lines of the file:
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@@
+	)
+	(gr_rect
+		(start 158.4965 40.1)
+		(end 178.0035 43)
+		(stroke
+			(width 0.1)
+			(type default)
+		)
+		(fill no)
+		(layer "F.SilkS")
 	)
 	(gr_rect
@@
 			)
 			(justify left bottom)
+		)
+	)
+	(gr_text "RTDS-Precharge | H.R. Oct '28"
+		(at 159 42.5 0)
+		(layer "F.SilkS")
+		(effects
+			(font
+				(size 1.5 0.75)
+				(thickness 0.1875)
+				(bold yes)
+			)
+			(justify left bottom)

Commit message: changes
changes
Other:
- board text added: "RTDS-Precharge | H.R. Oct '28 2025"
- board text removed: "RTDS-Precharge | H.R. Oct '28"
Changed lines of the file:
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@@
 	)
 	(gr_rect
-		(start 158.4965 40.1)
-		(end 178.0035 43)
+		(start 157 40.1)
+		(end 179.507 43.5)
 		(stroke
 			(width 0.1)
-			(type default)
+			(type solid)
 		)
 		(fill no)
@@
 		)
 	)
-	(gr_text "RTDS-Precharge | H.R. Oct '28"
-		(at 159 42.5 0)
+	(gr_text "RTDS-Precharge | H.R. Oct '28 2025"
+		(at 157 42.5 0)
 		(layer "F.SilkS")
 		(effects

Commit message: traces
traces
Routing:
- net Net-(U1-VCC): track 86.3 -> 66.7 mm, vias 1 -> 0
- net Net-(U6-TR): track 49.3 -> 67.7 mm, vias 1 -> 3
- net Net-(U6-GND): track 113.0 -> 130.1 mm, vias 0 -> 2
- net Net-(Q1-B): track 28.2 -> 16.2 mm
- net Net-(U6-VCC): track 87.5 -> 96.8 mm, vias 2 -> 1
- net Net-(U1-CV): track 24.3 -> 17.5 mm
- net Net-(U3-D): track 26.3 -> 19.7 mm, vias 1 -> 0
- net Net-(Q1-C): track 95.9 -> 102.5 mm, vias 3 -> 1
- net Net-(D3-A): track 57.0 -> 50.5 mm, vias 3 -> 2
- net Net-(D3-K): track 25.3 -> 19.2 mm, vias 1 -> 0
- net Net-(D2-K): track 26.0 -> 31.2 mm
- net Net-(Q1-E): track 27.4 -> 32.0 mm
- net Net-(J1-Pad9): track 16.6 -> 12.1 mm
- net Net-(U6-DIS): track 50.0 -> 54.4 mm
- net Net-(U6-CV): track 29.6 -> 26.2 mm
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