File: VCUThrottleLatching/VCUThrottleLatching.kicad_pcb (KiCad board)
At the start: 2 copper layers, 51 x 39.5 mm, 9 parts, among them J1 B12B-PH-K-S:JST_B12B-PH-K-S, U1 IRLML2060TRPBF, U2 IRLML2060TRPBF

Commit message: Silkscreen
silkscreen
Other:
- board text added: "VCU-ThrottleLatch | H.R. Oct '28"
Changed lines of the file:
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@@
+	)
+	(gr_rect
+		(start 133.7465 43.1)
+		(end 154.2535 46)
+		(stroke
+			(width 0.1)
+			(type default)
+		)
+		(fill no)
+		(layer "F.SilkS")
 	)
 	(gr_rect
@@
 		(layer "Edge.Cuts")
 	)
+	(gr_text "VCU-ThrottleLatch | H.R. Oct '28"
+		(at 134 45.5 0)
+		(layer "F.SilkS")
+		(effects
+			(font
+				(size 1.5 0.75)
+				(thickness 0.1875)
+				(bold yes)
+			)
+			(justify left bottom)
+		)
+	)
 	(gr_text "6: +5V                    4: GND\n5: From IMS/AMD Latch   3: VCU TL\n\n"

Commit message: changes
changes
Other:
- board text added: "VCU-ThrottleLatch | H.R. Oct '28 2025"
- board text removed: "VCU-ThrottleLatch | H.R. Oct '28"
Changed lines of the file:
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@@
 	)
 	(gr_rect
-		(start 133.7465 43.1)
-		(end 154.2535 46)
+		(start 132.2465 43.1)
+		(end 155.7535 46.5)
 		(stroke
 			(width 0.1)
@@
 		(layer "Edge.Cuts")
 	)
-	(gr_text "VCU-ThrottleLatch | H.R. Oct '28"
-		(at 134 45.5 0)
+	(gr_text "VCU-ThrottleLatch | H.R. Oct '28 2025"
+		(at 132.5 45.5 0)
 		(layer "F.SilkS")
 		(effects

Commit message: traces
traces
Routing:
- net Net-(D2-A): track 45.9 -> 33.5 mm, vias 0 -> 1
- net Net-(U2-G): track 27.0 -> 36.6 mm
- net Net-(D1-A): track 18.7 -> 14.3 mm, vias 2 -> 0
- net Net-(U1-G): track 31.9 -> 36.1 mm, vias 0 -> 1
- net Net-(U1-D): track 14.0 -> 16.0 mm, vias 0 -> 1
- net Net-(D1-K): track 14.9 -> 16.2 mm
- net Net-(U2-D): track 13.9 -> 14.2 mm, vias 1 -> 2
