File: LVChargeNEW/LVChargeNEW.kicad_pcb (KiCad board)
At the start: 2 copper layers, 41 parts, among them Q1 CSD15380F3T, Q2 CSD15380F3T, Q3 CSD15380F3T, Q4 CSD15380F3T, U1 PQ25856QWRRVRQ1

Commit message: LVCharge mostly done
Parts:
- added R12: 249k, Resistor_THT:R_Axial_DIN0204_L3.6mm_D1.6mm_P5.08mm_Horizontal, F.Cu at (88.9, 94.0)
- added R_bat_ac1: .005, LVChargeNEWLocalFootprints:RESC2012X80N, F.Cu at (116.8, 101.6)
- added R_bat_sns1: .005, LVChargeNEWLocalFootprints:RESC2012X80N, F.Cu at (98.1, 121.9)
- Q1, Q2, Q3, Q4: footprint LVChargeNEWLocalFootprints:CSD15380F3 -> LVChargeNEWLocalFootprints:IAUZ20N08S5L300ATMA1
- moved C1 34.7 mm to (73.6, 63.5), turned to 180 degrees
- moved C6 27.8 mm to (68.6, 104.1), turned to 90 degrees
- moved C8 27.1 mm to (73.7, 88.9), turned to 180 degrees
- moved C5 19.2 mm to (68.7, 78.7)
- moved Q2 19.2 mm to (124.5, 102.3), turned to 90 degrees
- moved Q1 16.0 mm to (121.9, 109.2), turned to 90 degrees
- moved Q4 7.40 mm to (142.2, 121.9), turned to 0 degrees
- moved Q3 6.69 mm to (159.3, 104.1), turned to 0 degrees
Connections:
- Q1 pad 1: Net-(U1-HIDRV1) -> Net-(U1-SW1)
- Q2 pad 1: Net-(U1-LODRV1) -> Batt-
- Q3 pad 1: Net-(U1-LODRV2) -> Net-(U1-SW2)
- Q4 pad 1: Net-(U1-HIDRV2) -> Batt-
Routing:
- net Buck Input: track 24.0 -> 153.4 mm, vias 0 -> 1
- net Batt-: track 309.9 -> 416.0 mm
- net Net-(U1-ACP): track 5.21 -> 106.6 mm
- net Net-(U1-ACN): track 118.1 -> 194.4 mm, vias 1 -> 2
- net Batt+: track 7.62 -> 49.7 mm, vias 0 -> 1
- net Net-(C9-Pad2): track 32.5 -> 73.8 mm, vias 2 -> 4
- net Net-(C12-Pad2): track 48.5 -> 76.1 mm, vias 1 -> 3
- net Net-(U1-SW1): track 238.8 -> 260.3 mm, vias 0 -> 3
- net Net-(U1-LODRV2): track 76.7 -> 57.7 mm
- net Net-(U1-FB): track 8.27 -> 26.7 mm, vias 0 -> 1
- net Net-(U1-HIDRV1): track 84.5 -> 102.1 mm
- net Net-(U1-BTST1): track 103.6 -> 92.0 mm
- net Net-(U1-HIDRV2): track 107.2 -> 97.7 mm
- net Net-(U1-LODRV1): track 102.3 -> 94.8 mm, vias 0 -> 2
- net Net-(U1-SW2): track 190.8 -> 197.7 mm
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