File: LVChargeNEW/_autosave-LVChargeNEW.kicad_sch (KiCad schematic)
At the start: 45 parts, among them Q1 CSD15380F3T, Q2 CSD15380F3T, Q3 CSD15380F3T, Q4 CSD15380F3T, U1 PQ25856QWRRVRQ1

Commit message: LVCharge mostly done
Parts:
- R_bat_ac1, R_bat_sns1: footprint (none) -> LVChargeNEWLocalFootprints:RESC2012X80N
Changed lines of the file:
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@@
 			)
 		)
-		(property "Footprint" ""
+		(property "Footprint" "LVChargeNEWLocalFootprints:RESC2012X80N"
 			(at 318.77 46.228 90)
 			(effects
@@
 			)
 		)
-		(property "Footprint" ""
+		(property "Footprint" "LVChargeNEWLocalFootprints:RESC2012X80N"
 			(at 109.728 99.06 90)
 			(effects
