File: Traces/Traces V1.0/Traces V1.0-DESKTOP-8S7ER7C.kicad_sch (KiCad schematic)
At the start: 3 parts, among them J1 B15B-PH-K-S, J2 B15B-PH-K-S, J3 B15B-PH-K-S

Commit message: Revert "changes"
This reverts commit 10df18be739a6716873fb9f13ef638a2302d6145.
Parts:
- added J4: B12B-PH-K-S, CONN12_B12B-PH_JST, symbol JST_PS_12pins:B12B-PH-K-S
Other:
- note added: "5V+ supply"
- note added: "AMS - 5V"
- note added: "AMSCC"
- note added: "GND"
- note added: "Reset +"
- note added: "Reset -"
- note added: "Safety Loop"
Changed lines of the file:
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@@
+		)
+	)
+	(text "5V+ supply"
+		(exclude_from_sim no)
+		(at 127.508 19.05 90)
+		(effects
+			(font
+				(size 0.762 0.762)
+			)
 		)
 	)
@@
 		)
 	)
+	(text "Vs"
+		(exclude_from_sim no)
+		(at 119.38 19.05 90)
+		(effects
+			(font
+				(size 0.762 0.762)
+			)
+		)
+	)
+	(text "Reset -"
+		(exclude_from_sim no)
+		(at 101.6 19.05 90)
+		(effects
+			(font
+				(size 0.762 0.762)
+			)
+		)
+	)
 	(text "Unused"
 		(exclude_from_sim no)
@@
 		)
 	)
+	(text "Safety Loop"
+		(exclude_from_sim no)
+		(at 114.808 19.05 90)
+		(effects
+			(font
+				(size 0.762 0.762)
+			)
+		)
+	)
 	(text "Unused"
 		(exclude_from_sim no)
@@
 		)
 	)
+	(text "5V+ supply"
+		(exclude_from_sim no)
+		(at 124.714 18.796 90)
+		(effects
+			(font
+				(size 0.762 0.762)
+			)
+		)
+	)
 	(text "AMS Reset +"
 		(exclude_from_sim no)
@@
 		)
 	)
+	(text "AMSCC"
+		(exclude_from_sim no)
+		(at 109.22 18.796 90)
+		(effects
+			(font
+				(size 0.762 0.762)
+			)
+		)
+	)
 	(text "Unused"
 		(exclude_from_sim no)
@@
 		)
 	)
+	(text "AMS LED +"
+		(exclude_from_sim no)
+		(at 107.188 18.288 90)
+		(effects
+			(font
+				(size 0.635 0.635)
+			)
+		)
+	)
+	(text "GND"
+		(exclude_from_sim no)
+		(at 111.76 18.796 90)
+		(effects
+			(font
+				(size 0.762 0.762)
+			)
+		)
+	)
 	(text "Unused"
 		(exclude_from_sim no)
@@
 		)
 	)
+	(text "AMS - 5V\n"
+		(exclude_from_sim no)
+		(at 113.284 14.478 0)
+		(effects
+			(font
+				(size 2.032 2.032)
+				(thickness 0.4064)
+				(bold yes)
+			)
+		)
+	)
+	(text "5V+ supply"
+		(exclude_from_sim no)
+		(at 121.92 18.796 90)
+		(effects
+			(font
+				(size 0.762 0.762)
+			)
+		)
+	)
 	(text "Unused"
 		(exclude_from_sim no)
@@
 		)
 	)
+	(text "GND\n"
+		(exclude_from_sim no)
+		(at 117.348 19.05 90)
+		(effects
+			(font
+				(size 0.762 0.762)
+			)
+		)
+	)
 	(text "TSMS Vs"
 		(exclude_from_sim no)
@@
 		)
 	)
+	(text "Vs"
+		(exclude_from_sim no)
+		(at 104.394 19.05 90)
+		(effects
+			(font
+				(size 0.762 0.762)
+			)
+		)
+	)
 	(text "VCU MPRD"
 		(exclude_from_sim no)
@@
 			(font
 				(size 1.27 1.27)
+			)
+		)
+	)
+	(text "Reset +"
+		(exclude_from_sim no)
+		(at 99.06 19.05 90)
+		(effects
+			(font
+				(size 0.762 0.762)
 			)
 		)
@@
 					(unit 1)
 				)
+			)
+		)
+	)
+	(symbol
+		(lib_id "JST_PS_12pins:B12B-PH-K-S")
+		(at 99.06 35.56 90)
+		(unit 1)
+		(exclude_from_sim no)
+		(in_bom yes)
+		(on_board yes)
+		(dnp no)
+		(property "Reference" "J4"
+			(at 90.17 35.814 0)
+			(effects
+				(font
+					(size 1.524 1.524)
+				)
+				(justify left)
+			)
+		)
+		(property "Value" "B12B-PH-K-S"
+			(at 93.472 35.306 0)
+			(effects
+				(font
+					(size 1.524 1.524)
+				)
+				(justify left)
+			)
+		)
+		(property "Footprint" "CONN12_B12B-PH_JST"
+			(at 99.06 35.56 0)
+			(effects
+				(font
+					(size 1.27 1.27)
+					(italic yes)
+				)
+				(hide yes)
+			)
+		)
+		(property "Datasheet" "B12B-PH-K-S"
+			(at 99.06 35.56 0)
+			(effects
+				(font
+					(size 1.27 1.27)
+					(italic yes)
+				)
+				(hide yes)
+			)
+		)
+		(property "Description" ""
+			(at 99.06 35.56 0)
+			(effects
+				(font
+					(size 1.27 1.27)
+				)
+				(hide yes)
+			)
+		)
+		(pin "5"
+		)
+		(pin "2"
+		)
+		(pin "1"
+		)
+		(pin "3"
+		)
+		(pin "4"
+		)
+		(pin "8"
+		)
+		(pin "9"
+		)
+		(pin "6"
+		)
+		(pin "10"
+		)
+		(pin "7"
+		)
+		(pin "12"
+		)
+		(pin "11"
+		)
+		(instances
+			(project "Traces V1.0"
+				(path "/2b8eb838-ed17-49da-bb42-10b70dc86c5e"
+					(reference "J4")
+					(unit 1)
+				)
