File: New LV Board/VCU Signals/VCU Signals.kicad_pcb (KiCad board)
At the start: 2 copper layers, 46 x 51.3 mm, 15 parts, among them J1 B12B-PH-K-S:JST_B12B-PH-K-S, P1 PH1-20-UA, P2 PH1-20-UA, U1 IRLML2060TRPBF, U2 IRLML2060TRPBF, U3 IRLML2060TRPBF

Commit message: fixed some silkscreen issues
Other:
- board text added: "VCU Signals | J.E. Nov 2025"
- board text removed: "VCU-ThrottleLatch | J.E. Nov 2025"
Changed lines of the file:
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@@
 	)
 	(gr_rect
-		(start 83.6914 77.7258)
+		(start 83.5136 77.7258)
 		(end 108.7882 81.1258)
 		(stroke
@@
 	)
 	(gr_text "PC Status - 1\nFrom PC - 2\nVCU Throttle Latch - 3\nFrom Saftey Loop - 4"
-		(at 108.2802 89.0524 0)
+		(at 108.2802 88.927899 0)
 		(layer "F.SilkS")
 		(effects
@@
 		)
 	)
-	(gr_text "VCU-ThrottleLatch | J.E. Nov 2025"
-		(at 85.344 80.41645 0)
+	(gr_text "VCU Signals | J.E. Nov 2025"
+		(at 87.587506 80.41645 0)
 		(layer "F.SilkS")
 		(effects
@@
 	)
 	(gr_text "8 - 5V\n7 - GND\n6 - From Charge Enable\n5 - VCU Charge Enable"
-		(at 83.7946 88.9 0)
+		(at 83.7946 88.927899 0)
 		(layer "F.SilkS")
 		(effects
@@
 	)
 	(gr_text "PINOUT"
-		(at 94.996 84.0232 0)
+		(at 93.275409 84.0232 0)
 		(layer "F.SilkS")
 		(effects
