File: New LV Board/IMD & AMS Latches/IMD & AMS Latches V1.0/IMD & AMS Latches V1.1.kicad_pcb (KiCad board)
At the start: 2 copper layers, 46 x 51.3 mm, 23 parts, among them J2 B12B-PH-K-S, K1 A161CS12VDC.64, K2 A161CS12VDC.64, K3 A161CS12VDC.64, K4 A161CS12VDC.64, K5 A161CS12VDC.64, K6 A161CS12VDC.64, P1 PH1-20-UA, P2 PH1-20-UA, SW1 Test Reset IMD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

Commit message: AMS & IMD fixing some connections
Parts:
- removed D3: 1N4001, Diode_THT:D_DO-41_SOD81_P10.16mm_Horizontal
- removed D5, D6: 1N4743A, motorsports:D_DO-41_SOD81_P3.81mm_Vertical_AnodeUp
- moved D2 6.57 mm to (99.7, 49.5)
- moved D1 4.34 mm to (99.7, 55.0)
Connections:
- K3 pad COM: Net-(J2-Pad4) -> Net-(J2-Pad2)
Routing:
- net Net-(D4-A): track 39.0 -> 77.2 mm
- net Net-(J2-Pad12): track 70.5 -> 40.4 mm
- net Net-(D8-A): track 92.7 -> 63.2 mm
- net Net-(D7-K): track 136.2 -> 107.9 mm
- net Net-(D1-A): track 116.9 -> 100.5 mm
- net Net-(J2-Pad1): track 8.09 -> 19.3 mm
- net Net-(J2-Pad2): track 69.6 -> 74.9 mm
- net Net-(D7-A): track 66.9 -> 63.1 mm
- net Net-(J2-Pad4): track 49.8 -> 46.5 mm
- net Net-(D1-K): track 79.5 -> 81.2 mm
Other:
- board text added: "AMS & IMD Latches V1.1 | J.W. Nov 2025"
- board text removed: "AMS & IMD Latches V1.0 | J.W. Nov 2025"
