File: New LV Board/Traces/Traces V1.0/Traces V1.0.kicad_pcb (KiCad board)
At the start: 2 copper layers, 105.7 x 51.8 mm, 15 parts, among them J1 B15B-PH-K-S, J2 B15B-PH-K-S, J3 B15B-PH-K-S, J4 Conn_01x12, J6 Conn_01x12, J7 Conn_01x12

Commit message: Traces Board Trace Makeover
Traces Board Trace Makeover
Routing:
- net Net-(J4-Pin_5): track 0.00 -> 159.0 mm
- net Net-(D2-K): track 0.00 -> 141.7 mm
- net Net-(J4-Pin_8): track 73.1 -> 200.2 mm
- net Net-(J6-Pin_11): track 0.00 -> 91.9 mm
- net Net-(J6-Pin_6): track 0.00 -> 86.5 mm
- net Net-(J6-Pin_10): track 0.00 -> 84.0 mm
- net Net-(D2-A): track 87.3 -> 168.9 mm
- net Net-(J6-Pin_12): track 35.3 -> 116.4 mm
- net Net-(J6-Pin_4): track 0.00 -> 80.6 mm
- net Net-(J6-Pin_5): track 0.00 -> 79.1 mm
- net Net-(J6-Pin_7): track 0.00 -> 72.5 mm
- net Net-(J6-Pin_8): track 0.00 -> 71.6 mm
- net Net-(J6-Pin_9): track 0.00 -> 68.8 mm
- net Net-(J4-Pin_1): track 0.00 -> 59.9 mm
- net Net-(J4-Pin_10): track 34.5 -> 80.7 mm
Other:
- copper layers 2 -> 6

Commit message: traces probably
Parts:
- added J5: B12B-PH-K-S, Connector_JST:JST_PH_B12B-PH-K_1x12_P2.00mm_Vertical, F.Cu at (116.8, 104.1)
- J1, J2, J3: footprint motorsports:JST_B15B-PH-K-S -> Connector_JST:JST_PH_B15B-PH-K_1x15_P2.00mm_Vertical
- J4, J6, J7: value Conn_01x12 -> B12B-PH-K-S; footprint motorsports:JST_B12B-PH-K-S -> Connector_JST:JST_PH_B12B-PH-K_1x12_P2.00mm_Vertical
- moved J6 70.3 mm to (41.9, 64.8)
- moved J4 37.9 mm to (92.7, 64.8)
- moved J7 22.5 mm to (66.0, 104.1), turned to 0 degrees
- moved J2 16.3 mm to (76.2, 99.2), turned to 90 degrees
- moved J3 10.9 mm to (53.3, 98.7), turned to 90 degrees
- moved J1 10.9 mm to (43.2, 98.7), turned to 90 degrees
- moved REF** 1.28 mm to (91.4, 61.0)
- moved REF** 1.28 mm to (91.4, 109.2)
Connections:
- F1 pad 3: Net-(J4-Pin_8) -> Net-(J4-Pin_5)
- F1 pad 4: Net-(J4-Pin_8) -> Net-(J4-Pin_5)
- J1 pad 1: Net-(J6-Pin_11) -> Net-(J6-Pin_8)
- J1 pad 10: Net-(J6-Pin_8) -> Net-(J1-Pad10)
- J1 pad 11: Net-(J6-Pin_9) -> Net-(J7-Pin_2)
- J1 pad 12: Net-(J6-Pin_7) -> Net-(J1-Pad10)
- J1 pad 13: Net-(J6-Pin_6) -> Net-(J6-Pin_1)
- J1 pad 14: Net-(J6-Pin_4) -> Net-(J4-Pin_1)
- J1 pad 15: Net-(J6-Pin_5) -> Net-(J6-Pin_2)
- J1 pad 2: Net-(J4-Pin_10) -> Net-(J6-Pin_9)
- J1 pad 3: Net-(J6-Pin_12) -> Net-(J6-Pin_7)
- J1 pad 4: unconnected-(J1-Pad4) -> Net-(J6-Pin_6)
- J1 pad 5: unconnected-(J1-Pad5) -> Net-(J6-Pin_4)
- J1 pad 6: unconnected-(J1-Pad6) -> Net-(J6-Pin_5)
- J1 pad 7: Net-(J7-Pin_11) -> Net-(J6-Pin_3)
- J1 pad 8: Net-(J4-Pin_1) -> Net-(J4-Pin_12)
- J1 pad 9: Net-(J6-Pin_10) -> Net-(J7-Pin_11)
- J2 pad 1: unconnected-(J2-Pad1) -> Net-(J7-Pin_3)
- J2 pad 2: unconnected-(J2-Pad2) -> Net-(J7-Pin_4)
- J2 pad 5: unconnected-(J2-Pad5) -> Net-(J5-Pin_9)
- J2 pad 6: unconnected-(J2-Pad6) -> Net-(J5-Pin_8)
- J2 pad 7: unconnected-(J2-Pad7) -> Net-(J5-Pin_7)
- J2 pad 8: unconnected-(J2-Pad8) -> Net-(J5-Pin_6)
- J3 pad 1: Net-(J4-Pin_5) -> Net-(D2-A)
- J3 pad 10: Net-(J4-Pin_5) -> Net-(J7-Pin_10)
- J3 pad 11: Net-(D2-K) -> Net-(J7-Pin_12)
- J3 pad 12: Net-(D2-K) -> Net-(J4-Pin_5)
- J3 pad 13: Net-(D2-K) -> unconnected-(J3-Pad13)
- J3 pad 14: Net-(D2-A) -> unconnected-(J3-Pad14)
- J3 pad 15: Net-(D2-A) -> Net-(J4-Pin_6)
- J3 pad 2: unconnected-(J3-Pad2) -> Net-(D2-A)
- J3 pad 3: unconnected-(J3-Pad3) -> Net-(D2-K)
- J3 pad 4: Net-(J4-Pin_8) -> Net-(D2-K)
- J3 pad 5: Net-(J7-Pin_12) -> Net-(D2-K)
- J3 pad 6: Net-(J7-Pin_10) -> Net-(J4-Pin_6)
- J3 pad 7: Net-(J7-Pin_8) -> Net-(J4-Pin_6)
- J3 pad 9: Net-(J4-Pin_5) -> Net-(J7-Pin_8)
- J4 pad 10: Net-(J4-Pin_10) -> Net-(D2-K)
- J4 pad 11: Net-(J4-Pin_10) -> Net-(D2-K)
- J4 pad 12: Net-(J4-Pin_10) -> Net-(J4-Pin_12)
- J4 pad 2: Net-(D2-K) -> Net-(J4-Pin_1)
- J4 pad 3: Net-(D2-K) -> Net-(J4-Pin_1)
- J4 pad 4: Net-(D2-K) -> Net-(D2-A)
- J4 pad 6: Net-(J4-Pin_5) -> Net-(J4-Pin_6)
- J4 pad 7: Net-(J4-Pin_5) -> Net-(J4-Pin_6)
- J4 pad 8: Net-(J4-Pin_8) -> Net-(J4-Pin_6)
- J4 pad 9: Net-(D2-A) -> Net-(D2-K)
- J6 pad 1: Net-(J4-Pin_5) -> Net-(J6-Pin_1)
- J6 pad 10: Net-(J6-Pin_10) -> Net-(D2-A)
- J6 pad 11: Net-(J6-Pin_11) -> Net-(J4-Pin_5)
- J6 pad 12: Net-(J6-Pin_12) -> Net-(J4-Pin_6)
- J6 pad 2: Net-(J4-Pin_8) -> Net-(J6-Pin_2)
- J6 pad 3: Net-(D2-A) -> Net-(J6-Pin_3)
- J7 pad 2: unconnected-(J7-Pin_2-Pad2) -> Net-(J7-Pin_2)
- J7 pad 3: unconnected-(J7-Pin_3-Pad3) -> Net-(J7-Pin_3)
- J7 pad 4: unconnected-(J7-Pin_4-Pad4) -> Net-(J7-Pin_4)
- J7 pad 5: Net-(J4-Pin_10) -> Net-(J4-Pin_1)
- J7 pad 9: Net-(J6-Pin_12) -> Net-(J6-Pin_1)
Routing:
- net Net-(J4-Pin_8): track 200.2 -> 0.00 mm, vias 1 -> 0
- net Net-(J4-Pin_5): track 159.0 -> 0.00 mm
- net Net-(D2-A): track 168.9 -> 35.7 mm, vias 1 -> 0
- net Net-(J6-Pin_12): track 116.4 -> 0.00 mm
- net Net-(J7-Pin_8): track 102.4 -> 0.00 mm
- net Net-(J7-Pin_7): track 97.8 -> 0.00 mm
- net Net-(D2-K): track 141.7 -> 46.6 mm
- net Net-(J6-Pin_11): track 91.9 -> 0.00 mm
- net Net-(J4-Pin_12): track 0.00 -> 85.7 mm
- net Net-(J6-Pin_10): track 84.0 -> 0.00 mm
- net Net-(J4-Pin_10): track 80.7 -> 0.00 mm
- net Net-(J7-Pin_12): track 56.2 -> 0.00 mm
- net Net-(J6-Pin_6): track 86.5 -> 31.6 mm
- net Net-(J7-Pin_10): track 52.8 -> 0.00 mm
- net Net-(J6-Pin_5): track 79.1 -> 26.8 mm, vias 0 -> 1
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Other:
- board size 105.7 x 51.8 mm -> 101.6 x 50.8 mm
- copper layers 6 -> 4

Commit message: traces
Parts:
- removed the REF** at (40.6, 61.0)
- removed the REF** at (40.6, 109.2)
- removed the REF** at (91.4, 61.0)
- removed TP3, TP4: TestPoint, TestPoint:TestPoint_Keystone_5005-5009_Compact
- added REF**: PinHeader_1x20_P2.54mm_Vertical, Connector_PinHeader_2.54mm:PinHeader_1x20_P2.54mm_Vertical, F.Cu at (91.4, 61.0)
- added REF**: PinHeader_1x20_P2.54mm_Vertical, Connector_PinHeader_2.54mm:PinHeader_1x20_P2.54mm_Vertical, F.Cu at (40.4, 61.0)
- added REF**: PinHeader_1x20_P2.54mm_Vertical, Connector_PinHeader_2.54mm:PinHeader_1x20_P2.54mm_Vertical, F.Cu at (40.3, 109.2)
- moved D2 37.8 mm to (55.5, 103.5), turned to -90 degrees
- moved C2 35.5 mm to (61.0, 103.5), turned to 90 degrees
- moved F1 29.9 mm to (65.5, 96.5), turned to 180 degrees
Routing:
- net Net-(J4-Pin_5): track 0.00 -> 210.0 mm, vias 0 -> 4
- net Net-(D2-A): track 35.7 -> 200.9 mm, vias 0 -> 2
- net Net-(J4-Pin_1): track 68.4 -> 181.7 mm, vias 0 -> 2
- net Net-(J4-Pin_6): track 44.6 -> 126.8 mm
- net Net-(J6-Pin_1): track 10.5 -> 89.7 mm, vias 0 -> 4
- net Net-(J5-Pin_9): track 0.00 -> 74.4 mm
- net Net-(D2-K): track 46.6 -> 120.8 mm, vias 0 -> 1
- net Net-(J7-Pin_12): track 0.00 -> 73.6 mm
- net Net-(J5-Pin_8): track 0.00 -> 72.0 mm
- net Net-(J7-Pin_10): track 0.00 -> 71.6 mm
- net Net-(J5-Pin_7): track 0.00 -> 70.1 mm
- net Net-(J5-Pin_6): track 0.00 -> 68.1 mm
- net Net-(J7-Pin_8): track 0.00 -> 44.7 mm
- net Net-(J7-Pin_7): track 0.00 -> 41.9 mm
- net Net-(J7-Pin_4): track 0.00 -> 26.3 mm
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Other:
- board text added: "1"
- board text added: "IMD & AMS Latches"
- board text added: "Potential Board"
- board text added: "Traces V2.0 | J.W. Feb 2026"
- board text added: "VCU MPR & 5V"
- board text added: "VCU Signals"
- board text removed: "J4"

Commit message: jlc
Other:
- copper layers 4 -> 2
Changed lines of the file:
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@@
 	(layers
 		(0 "F.Cu" signal)
-		(4 "In1.Cu" signal)
-		(6 "In2.Cu" signal)
 		(2 "B.Cu" signal)
 		(9 "F.Adhes" user "F.Adhesive")
@@
 			)
 			(layer "dielectric 1"
-				(type "prepreg")
-				(thickness 0.1)
+				(type "core")
+				(thickness 1.51)
 				(material "FR4")
 				(epsilon_r 4.5)
-				(loss_tangent 0.02)
-			)
-			(layer "In1.Cu"
-				(type "copper")
-				(thickness 0.035)
-			)
-			(layer "dielectric 2"
-				(type "core")
-				(thickness 1.24)
-				(material "FR4")
-				(epsilon_r 4.5)
-				(loss_tangent 0.02)
-			)
-			(layer "In2.Cu"
-				(type "copper")
-				(thickness 0.035)
-			)
-			(layer "dielectric 3"
-				(type "prepreg")
-				(thickness 0.1)
-				(material "FR4")
-				(epsilon_r 4.5)

Commit message: flipped connectors
Parts:
- moved J1 28.2 mm to (43.2, 70.5), turned to -90 degrees
- moved J2 28.1 mm to (76.2, 71.1), turned to -90 degrees
- moved J3 28.0 mm to (53.3, 70.7), turned to -90 degrees
- moved REF** 0.36 mm to (91.1, 109.2)
- moved REF** 0.34 mm to (91.1, 61.0)
- moved REF** 0.10 mm to (40.3, 61.0)
Connections:
- J2 pad 1: Net-(J7-Pin_3) -> unconnected-(J2-Pad15)
- J2 pad 10: unconnected-(J2-Pad10) -> Net-(J5-Pin_8)
- J2 pad 11: unconnected-(J2-Pad11) -> Net-(J5-Pin_9)
- J2 pad 14: unconnected-(J2-Pad14) -> Net-(J7-Pin_4)
- J2 pad 15: unconnected-(J2-Pad15) -> Net-(J7-Pin_3)
- J2 pad 2: Net-(J7-Pin_4) -> unconnected-(J2-Pad14)
- J2 pad 5: Net-(J5-Pin_9) -> unconnected-(J2-Pad11)
- J2 pad 6: Net-(J5-Pin_8) -> unconnected-(J2-Pad10)
- J2 pad 7: Net-(J5-Pin_7) -> unconnected-(J2-Pad9)
- J2 pad 9: unconnected-(J2-Pad9) -> Net-(J5-Pin_7)
- J3 pad 1: Net-(D2-A) -> Net-(J4-Pin_6)
- J3 pad 10: Net-(J7-Pin_10) -> Net-(J4-Pin_6)
- J3 pad 11: Net-(J7-Pin_12) -> Net-(D2-K)
- J3 pad 12: Net-(J4-Pin_5) -> Net-(D2-K)
- J3 pad 13: unconnected-(J3-Pad13) -> Net-(D2-K)
- J3 pad 14: unconnected-(J3-Pad14) -> Net-(D2-A)
- J3 pad 15: Net-(J4-Pin_6) -> Net-(D2-A)
- J3 pad 2: Net-(D2-A) -> unconnected-(J3-Pad14)
- J3 pad 3: Net-(D2-K) -> unconnected-(J3-Pad13)
- J3 pad 4: Net-(D2-K) -> Net-(J4-Pin_5)
- J3 pad 5: Net-(D2-K) -> Net-(J7-Pin_12)
- J3 pad 6: Net-(J4-Pin_6) -> Net-(J7-Pin_10)
- J3 pad 7: Net-(J4-Pin_6) -> Net-(J7-Pin_8)
- J3 pad 9: Net-(J7-Pin_8) -> Net-(J4-Pin_6)

Commit message: BANG
Connections:
- J2 pad 1: unconnected-(J2-Pad15) -> Net-(J7-Pin_3)
- J2 pad 10: Net-(J5-Pin_8) -> unconnected-(J2-Pad10)
- J2 pad 11: Net-(J5-Pin_9) -> unconnected-(J2-Pad11)
- J2 pad 14: Net-(J7-Pin_4) -> unconnected-(J2-Pad14)
- J2 pad 15: Net-(J7-Pin_3) -> unconnected-(J2-Pad15)
- J2 pad 2: unconnected-(J2-Pad14) -> Net-(J7-Pin_4)
- J2 pad 5: unconnected-(J2-Pad11) -> Net-(J5-Pin_9)
- J2 pad 6: unconnected-(J2-Pad10) -> Net-(J5-Pin_8)
- J2 pad 7: unconnected-(J2-Pad9) -> Net-(J5-Pin_7)
- J2 pad 9: Net-(J5-Pin_7) -> unconnected-(J2-Pad9)
- J3 pad 1: Net-(J4-Pin_6) -> Net-(D2-A)
- J3 pad 10: Net-(J4-Pin_6) -> Net-(J7-Pin_10)
- J3 pad 11: Net-(D2-K) -> Net-(J7-Pin_12)
- J3 pad 12: Net-(D2-K) -> Net-(J4-Pin_5)
- J3 pad 13: Net-(D2-K) -> unconnected-(J3-Pad13)
- J3 pad 14: Net-(D2-A) -> unconnected-(J3-Pad14)
- J3 pad 15: Net-(D2-A) -> Net-(J4-Pin_6)
- J3 pad 2: unconnected-(J3-Pad14) -> Net-(D2-A)
- J3 pad 3: unconnected-(J3-Pad13) -> Net-(D2-K)
- J3 pad 4: Net-(J4-Pin_5) -> Net-(D2-K)
- J3 pad 5: Net-(J7-Pin_12) -> Net-(D2-K)
- J3 pad 6: Net-(J7-Pin_10) -> Net-(J4-Pin_6)
- J3 pad 7: Net-(J7-Pin_8) -> Net-(J4-Pin_6)
- J3 pad 9: Net-(J4-Pin_6) -> Net-(J7-Pin_8)
Changed lines of the file:
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@@
 			(layers "*.Cu" "*.Mask")
 			(remove_unused_layers no)
-			(net 11 "unconnected-(J2-Pad15)")
-			(pinfunction "15")
+			(net 40 "Net-(J7-Pin_3)")
+			(pinfunction "1")
 			(pintype "passive")
 		)
@@
 			(layers "*.Cu" "*.Mask")
 			(remove_unused_layers no)
-			(net 8 "unconnected-(J2-Pad14)")
-			(pinfunction "14")
+			(net 38 "Net-(J7-Pin_4)")
+			(pinfunction "2")
 			(pintype "passive")
 		)
@@
 			(layers "*.Cu" "*.Mask")
 			(remove_unused_layers no)
-			(net 14 "unconnected-(J2-Pad13)")
-			(pinfunction "13")
+			(net 15 "unconnected-(J2-Pad3)")
+			(pinfunction "3")
 			(pintype "passive")
 		)
@@
 			(layers "*.Cu" "*.Mask")
 			(remove_unused_layers no)
-			(net 10 "unconnected-(J2-Pad12)")
-			(pinfunction "12")
+			(net 9 "unconnected-(J2-Pad4)")
+			(pinfunction "4")
 			(pintype "passive")
 		)
@@
 			(layers "*.Cu" "*.Mask")
 			(remove_unused_layers no)
-			(net 13 "unconnected-(J2-Pad11)")
-			(pinfunction "11")
+			(net 35 "Net-(J5-Pin_9)")
+			(pinfunction "5")
 			(pintype "passive")
 		)
@@
 			(layers "*.Cu" "*.Mask")
 			(remove_unused_layers no)
-			(net 12 "unconnected-(J2-Pad10)")
-			(pinfunction "10")
+			(net 36 "Net-(J5-Pin_8)")
+			(pinfunction "6")
 			(pintype "passive")
 		)
@@
 			(layers "*.Cu" "*.Mask")
 			(remove_unused_layers no)
-			(net 16 "unconnected-(J2-Pad9)")
-			(pinfunction "9")
+			(net 39 "Net-(J5-Pin_7)")
+			(pinfunction "7")
 			(pintype "passive")
 		)
@@
 			(layers "*.Cu" "*.Mask")
 			(remove_unused_layers no)
-			(net 39 "Net-(J5-Pin_7)")
-			(pinfunction "7")
+			(net 16 "unconnected-(J2-Pad9)")
+			(pinfunction "9")
 			(pintype "passive")
 		)
@@
 			(layers "*.Cu" "*.Mask")
 			(remove_unused_layers no)
-			(net 36 "Net-(J5-Pin_8)")
-			(pinfunction "6")
+			(net 12 "unconnected-(J2-Pad10)")
+			(pinfunction "10")
 			(pintype "passive")
 		)
@@
 			(layers "*.Cu" "*.Mask")
 			(remove_unused_layers no)
-			(net 35 "Net-(J5-Pin_9)")
-			(pinfunction "5")
+			(net 13 "unconnected-(J2-Pad11)")
+			(pinfunction "11")
 			(pintype "passive")
 		)
@@
 			(layers "*.Cu" "*.Mask")
 			(remove_unused_layers no)
-			(net 9 "unconnected-(J2-Pad4)")
-			(pinfunction "4")
+			(net 10 "unconnected-(J2-Pad12)")
+			(pinfunction "12")
 			(pintype "passive")
 		)
@@
 			(layers "*.Cu" "*.Mask")
 			(remove_unused_layers no)
-			(net 15 "unconnected-(J2-Pad3)")
-			(pinfunction "3")
+			(net 14 "unconnected-(J2-Pad13)")
+			(pinfunction "13")
 			(pintype "passive")
 		)
@@
 			(layers "*.Cu" "*.Mask")
 			(remove_unused_layers no)
-			(net 38 "Net-(J7-Pin_4)")
-			(pinfunction "2")
+			(net 8 "unconnected-(J2-Pad14)")
+			(pinfunction "14")
 			(pintype "passive")
 		)
@@
 			(remove_unused_layers no)
 			(roundrect_rratio 0.208333)
-			(net 40 "Net-(J7-Pin_3)")
-			(pinfunction "1")
+			(net 11 "unconnected-(J2-Pad15)")
+			(pinfunction "15")
 			(pintype "passive")
 		)
@@
 			(layers "*.Cu" "*.Mask")
 			(remove_unused_layers no)
-			(net 21 "Net-(J4-Pin_6)")
-			(pinfunction "15")
+			(net 19 "Net-(D2-A)")
+			(pinfunction "1")
 			(pintype "passive")
 		)
@@
 			(layers "*.Cu" "*.Mask")
 			(remove_unused_layers no)
-			(net 32 "unconnected-(J3-Pad14)")
-			(pinfunction "14")
+			(net 19 "Net-(D2-A)")
+			(pinfunction "2")
 			(pintype "passive")
 		)
@@
 			(layers "*.Cu" "*.Mask")
 			(remove_unused_layers no)
-			(net 31 "unconnected-(J3-Pad13)")
-			(pinfunction "13")
+			(net 18 "Net-(D2-K)")
+			(pinfunction "3")
 			(pintype "passive")
 		)
@@
 			(layers "*.Cu" "*.Mask")
 			(remove_unused_layers no)
-			(net 4 "Net-(J4-Pin_5)")
-			(pinfunction "12")
+			(net 18 "Net-(D2-K)")
+			(pinfunction "4")
 			(pintype "passive")
 		)
@@
 			(layers "*.Cu" "*.Mask")
 			(remove_unused_layers no)
-			(net 26 "Net-(J7-Pin_12)")
-			(pinfunction "11")
+			(net 18 "Net-(D2-K)")
+			(pinfunction "5")
 			(pintype "passive")
 		)
@@
 			(layers "*.Cu" "*.Mask")
 			(remove_unused_layers no)
-			(net 29 "Net-(J7-Pin_10)")
-			(pinfunction "10")
+			(net 21 "Net-(J4-Pin_6)")
+			(pinfunction "6")
 			(pintype "passive")
 		)
@@
 			(layers "*.Cu" "*.Mask")
 			(remove_unused_layers no)
-			(net 28 "Net-(J7-Pin_8)")
-			(pinfunction "9")
+			(net 21 "Net-(J4-Pin_6)")
+			(pinfunction "7")
 			(pintype "passive")
 		)
@@
 			(layers "*.Cu" "*.Mask")
 			(remove_unused_layers no)
-			(net 21 "Net-(J4-Pin_6)")
-			(pinfunction "7")
+			(net 28 "Net-(J7-Pin_8)")
+			(pinfunction "9")
 			(pintype "passive")
 		)
@@
 			(layers "*.Cu" "*.Mask")
 			(remove_unused_layers no)
-			(net 21 "Net-(J4-Pin_6)")
-			(pinfunction "6")
+			(net 29 "Net-(J7-Pin_10)")
+			(pinfunction "10")
 			(pintype "passive")
 		)
@@
 			(layers "*.Cu" "*.Mask")
 			(remove_unused_layers no)
-			(net 18 "Net-(D2-K)")
-			(pinfunction "5")
+			(net 26 "Net-(J7-Pin_12)")
+			(pinfunction "11")
 			(pintype "passive")
 		)
@@
 			(layers "*.Cu" "*.Mask")
 			(remove_unused_layers no)
-			(net 18 "Net-(D2-K)")
-			(pinfunction "4")
+			(net 4 "Net-(J4-Pin_5)")
+			(pinfunction "12")
 			(pintype "passive")
 		)
@@
 			(layers "*.Cu" "*.Mask")
 			(remove_unused_layers no)
-			(net 18 "Net-(D2-K)")
-			(pinfunction "3")
+			(net 31 "unconnected-(J3-Pad13)")
+			(pinfunction "13")
 			(pintype "passive")
 		)
@@
 			(layers "*.Cu" "*.Mask")
 			(remove_unused_layers no)
-			(net 19 "Net-(D2-A)")
-			(pinfunction "2")
+			(net 32 "unconnected-(J3-Pad14)")
+			(pinfunction "14")
 			(pintype "passive")
 		)
@@
 			(remove_unused_layers no)
 			(roundrect_rratio 0.208333)
-			(net 19 "Net-(D2-A)")
-			(pinfunction "1")
+			(net 21 "Net-(J4-Pin_6)")
+			(pinfunction "15")
 			(pintype "passive")
 		)
